Commit message: 修改雷达扫描范围不关于小车前方对称

File: sia_agv3/urdf/sia_717.urdf.xacro (robot description, xacro)
@@ -179,5 +179,5 @@
       name="${laser_name}_joint" type="fixed">
       <origin
-        xyz="0 0.67006 -0.529" rpy="0 0 0" />
+        xyz="0 0.67006 -0.529" rpy="0 0 1.57" />
       <parent
         link="base_link" />
@@ -189,5 +189,5 @@
         lower="-${PI}" upper="${PI}" effort="0" velocity="0" />
     </joint>
-</xacro:macro>
+  </xacro:macro>
   <link  name="base_link">
     <inertial>

File: sia_agv3/urdf/sia_laser.urdf.xacro (robot description, xacro)
@@ -11,6 +11,6 @@
             <samples>360</samples>
             <resolution>1</resolution>
-            <min_angle>-3</min_angle>
-            <max_angle>3</max_angle>
+            <min_angle>-2</min_angle>
+            <max_angle>2</max_angle>
           </horizontal>
         </scan>
