Commit message: update

File: sia_agv_description/urdf/sia_agv.urdf.xacro (robot description, xacro)
@@ -19,5 +19,5 @@
         <origin xyz="0 0 0" rpy="0 0 0" />
         <geometry>
-          <mesh filename="package://sia_agv3/meshes/agv_universal_wheel_hinge.dae" />
+          <mesh filename="package://sia_agv_description/meshes/agv_universal_wheel_hinge.dae" />
         </geometry>
       </visual>
@@ -42,5 +42,5 @@
         <origin xyz="0 0 0" rpy="0 0 0" />
         <geometry>
-          <mesh filename="package://sia_agv3/meshes/agv_universal_wheel_hinge.dae" />
+          <mesh filename="package://sia_agv_description/meshes/agv_universal_wheel_hinge.dae" />
         </geometry>
       </visual>
@@ -65,5 +65,5 @@
         <origin xyz="0 0 0" rpy="0 0 0" />
         <geometry>
-          <mesh filename="package://sia_agv3/meshes/agv_drive_wheel.dae" />
+          <mesh filename="package://sia_agv_description/meshes/agv_drive_wheel.dae" />
         </geometry>
         <material name="">
@@ -97,5 +97,5 @@
         <origin xyz="0 0 0" rpy="0 0 0" />
         <geometry>
-          <mesh filename="package://sia_agv3/meshes/agv_universal_wheel.dae" />
+          <mesh filename="package://sia_agv_description/meshes/agv_universal_wheel.dae" />
         </geometry>
       </visual>
@@ -126,5 +126,5 @@
         <origin xyz="0 0 0" rpy="0 0 0" />
         <geometry>
-          <mesh filename="package://sia_agv3/meshes/agv_laser_link.dae" />
+          <mesh filename="package://sia_agv_description/meshes/agv_laser_link.dae" />
         </geometry>
         <material name="">
@@ -150,5 +150,5 @@
       <origin xyz="0 0 0" rpy="0 0 0" />
       <geometry>
-        <mesh filename="package://sia_agv3/meshes/agv_base_link.dae" />
+        <mesh filename="package://sia_agv_description/meshes/agv_base_link.dae" />
       </geometry>
       <material name="">

Commit message: fix collisions

File: sia_agv_description/urdf/sia_agv.urdf.xacro (robot description, xacro)
@@ -158,7 +158,19 @@
     </visual>
     <collision>
+      <origin xyz="0 0.2765 -0.240" rpy="0 0 0" />
+      <geometry>
+        <box size="0.585 0.925 0.480" />
+      </geometry>
+    </collision>
+    <collision>
       <origin xyz="0 0 0" rpy="0 0 0" />
       <geometry>
-        <box size="0.925 0.585 0.67" />
+        <mesh filename="package://sia_agv_description/meshes/collisions/agv_base_link.stl" />
+      </geometry>
+    </collision>
+    <collision>
+      <origin xyz="0 0.2765 -0.5865" rpy="0 0 0" />
+      <geometry>
+        <box size="0.585 0.925 0.0525" />
       </geometry>
     </collision>

File: sia_agv_simulation/urdf/sia_laser.urdf.xacro (robot description, xacro)
@@ -11,6 +11,6 @@
             <samples>360</samples>
             <resolution>1</resolution>
-            <min_angle>-3</min_angle>
-            <max_angle>3</max_angle>
+            <min_angle>-0.5236</min_angle>
+            <max_angle>3.6652</max_angle>
           </horizontal>
         </scan>
