Commit message: 增添base_footprint

File: sia_agv_description/urdf/sia_agv_on_rviz.urdf.xacro (robot description, xacro)
@@ -134,5 +134,6 @@
     </link>
     <joint name="${laser_name}_joint" type="fixed">
-      <origin xyz="0 0.67006 -0.529" rpy="0 0 0" />
+      <origin xyz="0 0.67006 -0.529" rpy="0 0 1.5707" />
+       <!-- <origin xyz="0 0.67006 -0.529" rpy="0 0 1.5707" /> -->
       <parent link="base_link" />
       <child link="${laser_name}_link" />
@@ -187,3 +188,15 @@
   <xacro:universial_wheel_func wheel_name="left_rear" flag="-1" />
   <xacro:laser_func laser_name="laser" flag="-1" />
+  <link name="base_footprint">
+          <visual>
+              <geometry>
+                  <sphere radius="0.001" />
+              </geometry>
+          </visual>
+      </link>
+  <joint name="base_link2base_footprint" type="fixed">
+      <parent link="base_footprint" />
+      <child link="base_link"/>
+      <origin xyz="0 0 0.679"  rpy="0 0 -1.5707"/>
+  </joint>
 </robot>

Commit message: 增添试管架夹持机构，但是夹持机构在gazebo中自然滑动，暂存一个版本，修复中

File: sia_agv_description/urdf/sia_agv_on_rviz.urdf.xacro (robot description, xacro)
@@ -4,5 +4,6 @@
      For more information, please see http://wiki.ros.org/sw_urdf_exporter -->
 <robot xmlns:xacro="http://www.ros.org/wiki/xacro" name="sia_agv">
-  <xacro:property name="universial_wheel_radius" value="0.0325" />
+  <!-- <xacro:property name="universial_wheel_radius" value="0.0325" /> -->
+  <xacro:property name="universial_wheel_radius" value="0.033" />
   <xacro:property name="PI" value="3.1415926" />
   <xacro:property name="drive_wheel_radius" value="0.075" />
@@ -159,10 +160,10 @@
     </visual>
     <collision>
-      <origin xyz="0 0.2765 -0.240" rpy="0 0 0" />
-      <geometry>
-        <box size="0.585 0.925 0.480" />
-      </geometry>
-    </collision>
-    <collision>
+      <origin xyz="0 0.2765 -0.5865" rpy="0 0 0" />
+      <geometry>
+        <box size="0.585 0.925 0.0525" />
+      </geometry>
+    </collision>
+    <!-- <collision>
       <origin xyz="0 0 0" rpy="0 0 0" />
       <geometry>
@@ -175,5 +176,5 @@
         <box size="0.585 0.925 0.0525" />
       </geometry>
-    </collision>
+    </collision> -->
   </link>
   <xacro:bracket_func_front bracket_name_front="right_front" flag="1" />
@@ -200,3 +201,75 @@
       <origin xyz="0 0 0.679"  rpy="0 0 -1.5707"/>
   </joint> -->
+  <link name="base_link_tube">
+    <inertial>
+      <origin xyz="-0.014363760504454 0.0203917976213786 0.396202927097847" rpy="0 0 0" />
+      <mass value="4.68149593934385" />
+      <inertia
+        ixx="0.0242261061981686"
+        ixy="1.06389301348616E-05"
+        ixz="-0.000246359559055914"
+        iyy="0.0296477108535802"
+        iyz="-7.04189022538268E-05"
+        izz="0.00888940868288621" />
+    </inertial>
+    <visual>
+      <origin  xyz="0 0 0" rpy="0 0 0" />
+      <geometry>
+        <mesh filename="package://sia_agv_description/meshes/yidong/base_link.STL" />
+      </geometry>
+      <material
+        name="gray">
+        <color  rgba="0.898039215686275 0.917647058823529 0.929411764705882 1" />
+      </material>
+    </visual>
+    <collision>
+      <origin xyz="0 0 0"  rpy="0 0 0" />
+      <geometry>
+        <mesh filename="package://sia_agv_description/meshes/yidong/base_link.STL" />
+      </geometry>
+    </collision>
+  </link>
+  <link name="tube_link">
+    <inertial>
+      <origin xyz="4.9452E-05 -0.051238 0.034119"  rpy="0 0 0" />
+      <mass value="1.0714" />
+      <inertia
+        ixx="0.00065944"
+        ixy="5.7893E-11"
+        ixz="-6.1464E-08"
+        iyy="0.0025328"
+        iyz="-5.4851E-05"
+        izz="0.0026271" />
+    </inertial>
+    <visual>
+      <origin xyz="0 0 0"  rpy="0 0 0" />
+      <geometry>
+        <mesh filename="package://sia_agv_description/meshes/yidong/Empty_Link.STL" />
+      </geometry>
+      <material
+        name="gray">
+        <color  rgba="0.89804 0.91765 0.92941 1" />
+      </material>
+    </visual>
+    <collision>
+      <origin xyz="0 0 0"  rpy="0 0 0" />
+      <geometry>
+        <mesh filename="package://sia_agv_description/meshes/yidong/Empty_Link.STL" />
+      </geometry>
+    </collision>
+  </link>
+  <joint  name="base2base_link_tube_joint"  type="fixed">
+    <origin xyz="0.12 0.15 0.03"  rpy="0 0 3.1415" />
+    <parent  link="base_link" />
+    <child  link="base_link_tube" />
+    <axis  xyz="0 0 -1" />
+    <limit lower="-${PI}" upper="${PI}" effort="0" velocity="0" />
+  </joint>
+   <joint name="move_platform_joint"  type="prismatic">
+    <origin  xyz="-0.021579 -0.27516 0.047539"  rpy="0 0 0" />
+    <parent  link="base_link_tube" />
+    <child  link="tube_link" />
+    <axis xyz="0 1 0" />
+    <limit lower="-0.03" upper="0.06" effort="0" velocity="0" />
+  </joint>
 </robot>

File: sia_agv_simulation/urdf/sia_agv_controller.urdf.xacro (robot description, xacro)
@@ -68,4 +68,13 @@
         <maxVel>1.0</maxVel>
     </gazebo>
+   <gazebo reference="tube_link">
+        <mu1>10000</mu1>
+        <mu2>10000</mu2>
+        <kp>500000.0</kp>
+        <kd>10.0</kd>
+        <minDepth>0.001</minDepth>
+        <maxVel>0.1</maxVel>
+        <fdir1>1 0 0</fdir1>
+    </gazebo>
     <!-- 控制器 -->
     <gazebo>
@@ -91,5 +100,5 @@
             <odometryTopic>odom</odometryTopic>            <!-- 里程计话题 -->
             <publishOdomTF>true</publishOdomTF>
-            <robotBaseFrame>base_footprint</robotBaseFrame>            <!-- 根坐标系 -->
+            <robotBaseFrame>base_link</robotBaseFrame>            <!-- 根坐标系 base_footprint-->
         </plugin>
     </gazebo>
@@ -104,4 +113,7 @@
             <!-- <robotNamespace>/</robotNamespace> -->
             <jointName>
+<!--
+                base2base_link_tube_joint, -->
+                move_platform_joint,
                 right_front_joint,
                 right_front_wheel_joint,

File: sia_agv_simulation/urdf/sia_agv_gazebo.urdf.xacro (robot description, xacro)
@@ -2,4 +2,3 @@
     <xacro:include filename="$(find sia_agv_description)/urdf/sia_agv_on_rviz.urdf.xacro" />
     <xacro:include filename="$(find sia_agv_simulation)/urdf/sia_agv_controller.urdf.xacro" />
-    <!-- <xacro:include filename="$(find sia_agv_simulation)/urdf/sia_laser.urdf.xacro" /> -->
 </robot>

File: sia_robot_simulation/urdf/sia_robot_on_gazebo.xacro (robot description, xacro)
@@ -69,4 +69,12 @@
         <maxVel>1.0</maxVel>
     </gazebo>
+    <!-- <gazebo reference="yidong">
+        <mu1>0.1</mu1>
+        <mu2>0.1</mu2>
+        <kp>1000000.0</kp>
+        <kd>100.0</kd>
+        <minDepth>0.001</minDepth>
+        <maxVel>1.0</maxVel>
+    </gazebo> -->
     <xacro:macro name="joint_trans" params="joint_name">
         <transmission name="${joint_name}_trans">
