Commit message: 机械臂初稿

File: sia_manipulator_description/urdf/sia_robot.urdf.xacro (robot description, xacro)
@@ -1,918 +1,16 @@
-<?xml version="1.0" ?>
-<robot xmlns:xacro="http://www.ros.org/wiki/xacro"
- name="siasun_GCR10">
-<material name ="Blue">
-   <color rgba="0.137 0.49412 0.74902 1"/>
- </material>
-<material name ="Black">
-   <color rgba="0 0 0 0.8"/>
- </material>
-<material name ="Dark Blue">
-   <color rgba="0.098 0.098 0.439 1.0"/>
- </material>
-<material name ="light Blue">
-   <color rgba="0.387 0.584 0.93 1.0"/>
- </material>
-<material name ="White">
-   <color rgba="1 1 1 1"/>
- </material>
-<material name ="Antique White">
-   <color rgba="0.98 0.92 0.84 1"/>
- </material>
-<material name ="Dark Gray">
-   <color rgba="0.537 0.594 0.74902 1"/>
- </material>
-<material name ="Gray">
-   <color rgba="0.537 0.594 0.74 1"/>
- </material>
- <material name ="Silver">
-    <color rgba="0.588 0.588 0.588 1"/>
- </material>
- <material name ="Red">
-    <color rgba="1.00 0 0 1.0"/>
- </material>
-<link
-    name="base_link">
-    <inertial>
-      <origin
-        xyz="-0.000543863853506091 0.282716810863512 -0.36138635137112"
-        rpy="0 0 0" />
-      <mass
-        value="29.2907917401275" />
-      <inertia
-        ixx="0.658416147229005"
-        ixy="0.000444325594903029"
-        ixz="-5.22965035739952E-05"
-        iyy="0.481294666894637"
-        iyz="0.000150147215019541"
-        izz="0.989603236439599" />
-    </inertial>
-    <visual>
-      <origin
-        xyz="0 0 0"
-        rpy="0 0 0" />
-      <geometry>
-        <mesh
-          filename="package://sia_robot/meshes/agv_base_link.dae" />
-      </geometry>
-      <material
-        name="">
-        <color
-          rgba="1 1 1 1" />
-      </material>
-    </visual>
-    <collision>
-      <origin
-        xyz="0 0 0"
-        rpy="0 0 0" />
-      <geometry>
-        <box size="1 1 1" />
-      </geometry>
-    </collision>
-  </link>
-  <link
-    name="1_Link">
-    <inertial>
-      <origin
-        xyz="-8.14202632020283E-05 0.00610304740119338 -0.0161440698140209"
-        rpy="0 0 0" />
-      <mass
-        value="0.0728108307863773" />
-      <inertia
-        ixx="2.279226907759E-05"
-        ixy="-1.52431962880911E-07"
-        ixz="-1.17033639983441E-07"
-        iyy="2.43402166733781E-05"
-        iyz="1.19958125852891E-06"
-        izz="3.97943793169979E-05" />
-    </inertial>
-    <visual>
-      <origin
-        xyz="0 0 0"
-        rpy="0 0 0" />
-      <geometry>
-        <mesh
-          filename="package://sia_robot/meshes/agv_axis1.dae" />
-      </geometry>
-      <material
-        name="">
-        <color
-          rgba="1 1 0.501960784313725 1" />
-      </material>
-    </visual>
-    <collision>
-      <origin
-        xyz="0 0 0"
-        rpy="0 0 0" />
-      <geometry>
-        <mesh
-          filename="package://sia_robot/meshes/agv_axis1.dae" />
-      </geometry>
-    </collision>
-  </link>
-  <joint
-    name="1-joint"
-    type="continuous">
-    <origin
-      xyz="-0.194 0.59539 -0.604"
-      rpy="0 0 0" />
-    <parent
-      link="base_link" />
-    <child
-      link="1_Link" />
-    <axis
-      xyz="0 0 -1" />
-    <limit
-      lower="-3.14"
-      upper="3.14"
-      effort="0"
-      velocity="0" />
-  </joint>
-  <link
-    name="1-1_Link">
-    <inertial>
-      <origin
-        xyz="1.54128708518275E-07 -6.35365208223604E-07 -2.08668753956531E-07"
-        rpy="0 0 0" />
-      <mass
-        value="0.126066263473178" />
-      <inertia
-        ixx="3.69211700768695E-05"
-        ixy="1.59275080958781E-11"
-        ixz="-4.07947748521245E-10"
-        iyy="3.69211197129469E-05"
-        iyz="1.49202086216788E-09"
-        izz="6.47847031089787E-05" />
-    </inertial>
-    <visual>
-      <origin
-        xyz="0 0 0"
-        rpy="0 0 0" />
-      <geometry>
-        <mesh
-          filename="package://sia_robot/meshes/agv_universal_wheel.dae" />
-      </geometry>
-      <material
-        name="">
-        <color
-          rgba="1 1 0.501960784313725 1" />
-      </material>
-    </visual>
-    <collision>
-      <origin
-        xyz="0 0 0"
-        rpy="0 0 0" />
-      <geometry>
-        <mesh
-          filename="package://sia_robot/meshes/agv_universal_wheel.dae" />
-      </geometry>
-    </collision>
-  </link>
-  <joint
-    name="1-1_joint"
-    type="continuous">
-    <origin
-      xyz="-0.0019416 0.019905 -0.0435"
-      rpy="1.5708 0 -1.4736" />
-    <parent
-      link="1_Link" />
-    <child
-      link="1-1_Link" />
-    <axis
-      xyz="0 0 -1" />
-    <limit
-      lower="-3.14"
-      upper="3.14"
-      effort="0"
-      velocity="0" />
-  </joint>
-  <link
-    name="2_Link">
-    <inertial>
-      <origin
-        xyz="-0.000336543565982339 0.0067145336674802 -0.0138488838342261"
-        rpy="0 0 0" />
-      <mass
-        value="0.0773960442571589" />
-      <inertia
-        ixx="2.79271956658027E-05"
-        ixy="-2.09328673275462E-07"
-        ixz="-1.86296961191266E-07"
-        iyy="2.93597569308493E-05"
-        iyz="-2.80412358155225E-08"
-        izz="4.69036460817845E-05" />
-    </inertial>
-    <visual>
-      <origin
-        xyz="0 0 0"
-        rpy="0 0 0" />
-      <geometry>
-        <mesh
-          filename="package://sia_robot/meshes/agv_axis2.dae" />
-      </geometry>
-      <material
-        name="">
-        <color
-          rgba="0.854901960784314 0.854901960784314 0.854901960784314 1" />
-      </material>
-    </visual>
-    <collision>
-      <origin
-        xyz="0 0 0"
-        rpy="0 0 0" />
-      <geometry>
-        <mesh
-          filename="package://sia_robot/meshes/agv_axis2.dae" />
-      </geometry>
-    </collision>
-  </link>
-  <joint
-    name="2-joint"
-    type="continuous">
-    <origin
-      xyz="0.194 0.59535 -0.6056"
-      rpy="0 0 0" />
-    <parent
-      link="base_link" />
-    <child
-      link="2_Link" />
-    <axis
-      xyz="0 0 -1" />
-    <limit
-      lower="-3.14"
-      upper="3.14"
-      effort="0"
-      velocity="0" />
-  </joint>
-  <link
-    name="2-1_Link">
-    <inertial>
-      <origin
-        xyz="8.63289463803874E-08 -6.61745890639942E-07 2.14074135862496E-07"
-        rpy="0 0 0" />
-      <mass
-        value="0.126066298764299" />
-      <inertia
-        ixx="3.69211742911089E-05"
-        ixy="3.29619978086518E-12"
-        ixz="1.35062822981863E-10"
-        iyy="3.6921114726363E-05"
-        iyz="-1.54062454753047E-09"
-        izz="6.47847019668671E-05" />
-    </inertial>
-    <visual>
-      <origin
-        xyz="0 0 0"
-        rpy="0 0 0" />
-      <geometry>
-        <mesh
-          filename="package://sia_robot/meshes/agv_universal_wheel.dae" />
-      </geometry>
-      <material
-        name="">
-        <color
-          rgba="1 1 0.501960784313725 1" />
-      </material>
-    </visual>
-    <collision>
-      <origin
-        xyz="0 0 0"
-        rpy="0 0 0" />
-      <geometry>
-        <mesh
-          filename="package://sia_robot/meshes/agv_universal_wheel.dae" />
-      </geometry>
-    </collision>
-  </link>
-  <joint
-    name="2-1_joint"
-    type="continuous">
-    <origin
-      xyz="-0.0028411 0.022783 -0.042013"
-      rpy="1.5807 0.069104 -1.4279" />
-    <parent
-      link="2_Link" />
-    <child
-      link="2-1_Link" />
-    <axis
-      xyz="0 0 -1" />
-    <limit
-      lower="-3.14"
-      upper="3.14"
-      effort="0"
-      velocity="0" />
-  </joint>
-  <link
-    name="3_Link">
-    <inertial>
-      <origin
-        xyz="-6.93889390390723E-18 0 0.00168998379535312"
-        rpy="0 0 0" />
-      <mass
-        value="0.418358558488212" />
-      <inertia
-        ixx="0.000915617766712358"
-        ixy="3.32582077666032E-20"
-        ixz="1.88985288748301E-20"
-        iyy="0.000915617766712358"
-        iyz="-8.76135733408917E-21"
-        izz="0.00170660288564837" />
-    </inertial>
-    <visual>
-      <origin
-        xyz="0 0 0"
-        rpy="0 0 0" />
-      <geometry>
-        <mesh
-          filename="package://sia_robot/meshes/agv_drive_wheel.dae" />
-      </geometry>
-      <material
-        name="">
-        <color
-          rgba="1 1 0.501960784313725 1" />
-      </material>
-    </visual>
-    <collision>
-      <origin
-        xyz="0 0 0"
-        rpy="0 0 0" />
-      <geometry>
-        <mesh
-          filename="package://sia_robot/meshes/agv_drive_wheel.dae" />
-      </geometry>
-    </collision>
-  </link>
-  <joint
-    name="3_joint"
-    type="continuous">
-    <origin
-      xyz="-0.2595 0.2765 -0.605"
-      rpy="1.5708 0 -1.5708" />
-    <parent
-      link="base_link" />
-    <child
-      link="3_Link" />
-    <axis
-      xyz="0 0 -1" />
-    <limit
-      lower="-3.14"
-      upper="3.14"
-      effort="0"
-      velocity="0" />
-  </joint>
-  <link
-    name="4_Link">
-    <inertial>
-      <origin
-        xyz="6.12704331715008E-15 -4.79616346638068E-14 0.00282199284179585"
-        rpy="0 0 0" />
-      <mass
-        value="0.250538971616596" />
-      <inertia
-        ixx="0.000465816741663599"
-        ixy="5.65058656963556E-20"
-        ixz="3.31873042587156E-19"
-        iyy="0.000465816741663599"
-        iyz="-1.71216168600813E-20"
-        izz="0.000863128969172632" />
-    </inertial>
-    <visual>
-      <origin
-        xyz="0 0 0"
-        rpy="0 0 0" />
-      <geometry>
-        <mesh
-          filename="package://sia_robot/meshes/agv_drive_wheel.dae" />
-      </geometry>
-      <material
-        name="">
-        <color
-          rgba="1 1 0.501960784313725 1" />
-      </material>
-    </visual>
-    <collision>
-      <origin
-        xyz="0 0 0"
-        rpy="0 0 0" />
-      <geometry>
-        <mesh
-          filename="package://sia_robot/meshes/agv_drive_wheel.dae" />
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