Commit message: 移动文件位置

File: sia_manipulator_description/urdf/sia_manipulator.xacro (robot description, xacro)
@@ -2,6 +2,4 @@
 <robot xmlns:xacro="http://www.ros.org/wiki/xacro"
  name="sia_manipulator">
-  <xacro:include filename="$(find sia_manipulator_description)/urdf/sia.gazebo.xacro" />
-  <xacro:include filename="$(find sia_manipulator_description)/urdf/sia.transmission.xacro" />
   <material name ="Blue">
     <color rgba="0.137 0.49412 0.74902 1"/>
@@ -59,21 +57,21 @@
   <!-- shoulder -->
   <link name="shoulder">
-      <visual>
-        <origin rpy="0 0 0" xyz="0 0 0"/>
-        <geometry>
-          <mesh filename="package://sia_manipulator_description/meshes/link1.dae"/>
-        </geometry>
-        <material name ="Blue"/>
-      </visual>
-      <collision>
-        <origin rpy="0 0 0" xyz="0 0 0"/>
-        <geometry>
-          <mesh filename="package://sia_manipulator_description/meshes/link1.stl"/>
-        </geometry>
-      </collision>
-      <inertial>
-        <mass value="12.369"/>
-        <inertia ixx="0.069552066" ixy="0.000045456" ixz="0.000067368" iyy="0.0682463" iyz="0.000262322" izz="0.054371276"/>
-      </inertial>
+       <visual>
+      <origin rpy="0 0 0" xyz="0 0 0"/>
+      <geometry>
+        <mesh filename="package://sia_manipulator_description/meshes/link1.dae"/>
+      </geometry>
+      <material name ="Blue"/>
+    </visual>
+    <collision>
+      <origin rpy="0 0 0" xyz="0 0 0"/>
+      <geometry>
+        <mesh filename="package://sia_manipulator_description/meshes/link1.stl"/>
+      </geometry>
+    </collision>
+    <inertial>
+      <mass value="12.369"/>
+      <inertia ixx="0.069552066" ixy="0.000045456" ixz="0.000067368" iyy="0.0682463" iyz="0.000262322" izz="0.054371276"/>
+    </inertial>
     </link>
   <!-- shoulder_joint -->
@@ -234,5 +232,3 @@
       <limit effort="140.0" lower="${-pi}" upper="${pi}" velocity="${165*pi/180}"/>
     </joint>
-  <xacro:sia_gazebo  flag="-1"  />
-  <xacro:sia_arm_transmission  hw_interface="PositionJointInterface" />
 </robot>

Commit message: add manipulator's base.dae

File: sia_manipulator_description/urdf/sia_manipulator.xacro (robot description, xacro)
@@ -39,5 +39,5 @@
         <origin rpy="0 0 0" xyz="0 0 0"/>
         <geometry>
-          <mesh filename="package://sia_manipulator_description/meshes/base.stl"/>
+          <mesh filename="package://sia_manipulator_description/meshes/base.dae"/>
         </geometry>
         <material name ="Gray"/>

Commit message: 整合小车和机械臂的仿真模型，但是在gazebo仿真，小车不动，后续排查

File: sia_manipulator_description/urdf/sia_manipulator.xacro (robot description, xacro)
@@ -35,5 +35,6 @@
   <!-- base_link -->
   <!-- 存在问题，质量惯性矩阵？ -->
-    <link name="base_link">
+  <!-- 更改base_link为duoco_base_link 方便和小车连接-->
+    <link name="duco_base_link">
       <visual>
         <origin rpy="0 0 0" xyz="0 0 0"/>
@@ -78,5 +79,5 @@
   <joint name="shoulder_joint" type="revolute">
       <origin rpy="0 0 ${-pi/2}" xyz="0 0 0.165"/>
-      <parent link="base_link"/>
+      <parent link="duco_base_link"/>
       <child link="shoulder"/>
       <axis xyz="0 0 1"/>

File: sia_manipulator_simulation/urdf/sia_manipulator_gazebo.urdf.xacro (robot description, xacro)
@@ -15,5 +15,5 @@
   <joint name="world_joint" type="fixed">
     <parent link="world" />
-    <child link = "base_link" />
+    <child link = "duco_base_link" />
     <origin xyz="0.0 0.0 0.0" rpy="0.0 0.0 0.0" />
   </joint>
