Commit message: 替换.dae解决模型不在gazebo显示，但是仍缺少夹爪的力传感器，暂存版本

File: sia_manipulator_description/urdf/robotiq_arg2f.xacro (robot description, xacro)
@@ -2,5 +2,5 @@
 <robot xmlns:xacro="http://ros.org/wiki/xacro">
   <xacro:macro name="robotiq_arg2f_base_link" params="prefix">
-    <link name="${prefix}robotiq_arg2f_base_link">
+    <!-- <link name="${prefix}robotiq_arg2f_base_link">
       <inertial>
         <origin xyz="8.625E-08 -4.6583E-06 0.03145" rpy="0 0 0" />
@@ -23,5 +23,25 @@
         </geometry>
       </collision>
-    </link>
+    </link> -->
+    <link name="${prefix}robotiq_arg2f_base_link">
+      <visual>
+      <origin xyz="0 0 0" rpy="0 -1.5707 0" />
+                <geometry>
+                    <mesh filename="package://sia_manipulator_description/meshes/visual/robotiq_85_base_link.dae"/>
+                </geometry>
+            </visual>
+            <collision>
+                <geometry>
+                    <mesh filename="package://sia_manipulator_description/meshes/collision/robotiq_85_base_link.stl"/>
+                </geometry>
+            </collision>
+            <inertial>
+                <mass value="0.636951" />
+                <origin xyz="0.0 0.0 0.0" />
+                <inertia ixx = "0.000380" ixy = "0.000000" ixz = "0.000000"
+                         iyx = "0.000000" iyy = "0.001110" iyz = "0.000000"
+                         izx = "0.000000" izy = "0.000000" izz = "0.001171" />
+            </inertial>
+        </link>
   </xacro:macro>
   <xacro:macro name="finger_joints" params="prefix fingerprefix reflect">

File: sia_manipulator_description/urdf/sia_maipulator_with_force_sensor.xacro (robot description, xacro)
@@ -121,5 +121,5 @@
     </link>
     <joint name="gripper_connect_joint" type="fixed">
-        <origin xyz="0.0 0 0.014" rpy="0 0.0 0.0"/>
+        <origin xyz="0.0 0 0.014" rpy="0 0 0.0"/>
         <parent link="ft_sensor"/>
         <child link="gripper_connect"/>
@@ -128,5 +128,5 @@
     </joint>
     <joint name="gripper_connect" type="fixed">
-        <origin xyz="0.0 0 0.0501" rpy="0 0.0 0.0"/>
+        <origin xyz="0.0 0 0.0501" rpy="0 0 0.0"/>
         <parent link="gripper_connect"/>
         <child link="robotiq_arg2f_base_link"/>
