Commit message: 不稳定版本，存在错误，存档一下

File: sia_manipulator_description/urdf/sia_maipulator_with_force_sensor.xacro (robot description, xacro)
@@ -2,4 +2,9 @@
 <robot xmlns:xacro="http://wiki.ros.org/xacro"
        name="sia_manipulator_with_force_sensor" >
+  <xacro:arg name="use_nominal_extrinsics" default="true"/>
+  <xacro:include filename="$(find sia_manipulator_description)/urdf/_d455.urdf.xacro" />
+   <xacro:include filename="$(find sia_manipulator_description)/urdf/robotiq_arg2f_85_model_macro.xacro" />
+  <xacro:robotiq_arg2f_85 prefix=""/>
+    <xacro:include filename="$(find sia_manipulator_description)/urdf/depthcam.xacro"/>
   <xacro:include filename="$(find sia_manipulator_description)/urdf/sia_manipulator.xacro" />
    <xacro:property name="force_sensor_radius" value="0.0295" /> <!-- base_footprint 半径  -->
@@ -14,12 +19,95 @@
         </inertial>
     </xacro:macro>
-    <link name="ft_sensor">
+    <!-- 摄像头支架 -->
+    <link name="cammera_connect">
+        <!-- <inertial>
+        <origin xyz="-0.0 -0.0 0" rpy="0 0 0" />
+        <mass value="0.000232947101621511" />
+        <inertia
+            ixx="3.81432002620824E-07"
+            ixy="-3.80269042713563E-08"
+            ixz="6.9685808649034E-10"
+            iyy="2.34507884179749E-07"
+            iyz="2.88744525437204E-09"
+            izz="6.00940338038487E-07" />
+        </inertial> -->
         <visual>
+        <origin xyz="0 0 0" rpy="0 0 0.25" />
+        <geometry>
+            <mesh
+            filename="package://sia_manipulator_description/meshes/cammera_connect.STL" />
+        </geometry>
+        <material
+            name="">
+            <color rgba="1 1 0.501960784313725 1" />
+        </material>
+        </visual>
+        <collision>
             <geometry>
                 <cylinder radius="${force_sensor_radius}" length="${force_sensor_h}" />
             </geometry>
             <origin xyz="0.0 0.0 0.0" rpy="0 0.0 0.0"/>
+        </collision>
+        <xacro:cylinder_inertial_matrix m="${force_sensor_mass}" r="${force_sensor_radius}" h="${force_sensor_h}" />
+    </link>
+    <link name="ft_sensor">
+        <visual>
+            <geometry>
+        <mesh
+          filename="package://sia_manipulator_description/meshes/ft_sensor.STL" />
+      </geometry>
+            <origin xyz="0.0009 0.09 -0.001" rpy="0 0.0 0"/>
             <material name="yellow">
-                <color rgba="0.5 0.3 0.0 0.5" />
+                <color rgba="0.5 0.3 0.0 1" />
+            </material>
+        </visual>
+        <collision>
+            <geometry>
+                <cylinder radius="${force_sensor_radius}" length="${force_sensor_h}" />
+            </geometry>
+            <origin xyz="0.0 0.0 0.0" rpy="0 0.0 0.0"/>
+        </collision>
+        <inertial>
+            <origin
+                xyz="0 0 0" rpy="0 0 0" />
+            <mass
+                value="0.03" />
+            <inertia
+                ixx="1.50391235062321E-05"
+                ixy="-4.66673091890262E-08"
+                ixz="-1.64107101311957E-07"
+                iyy="2.97884994987516E-05"
+                iyz="5.6752026498067E-08"
+                izz="1.58243373451487E-05" />
+        </inertial>
+    </link>
+    <joint name="cammera_connect_joint" type="fixed">
+        <origin xyz="0.0 0 0.009" rpy="0 0.0 0.0"/>
+        <parent link="wrist_3"/>
+        <child link="cammera_connect"/>
+        <axis xyz="0.0 0.0 0.0"/>
+        <limit effort="140.0" lower="${-pi}" upper="${pi}" velocity="${165*pi/180}"/>
+    </joint>
+    <joint name="ft_sensor_joint" type="fixed">
+        <origin xyz="0.0 0 0" rpy="0 0.0 0.0"/>
+        <parent link="cammera_connect"/>
+        <child link="ft_sensor"/>
+        <axis xyz="0.0 0.0 0.0"/>
+        <limit effort="140.0" lower="${-pi}" upper="${pi}" velocity="${165*pi/180}"/>
+    </joint>
+    <!-- <xacro:sensor_d455 parent="cammera_connect" use_nominal_extrinsics="$(arg use_nominal_extrinsics)">
+    <origin xyz="0.001 -0.07 0.0175" rpy="1.5707 -1.5707 0"/>
+    </xacro:sensor_d455> -->
+    <xacro:realsense_d435 sensor_name="d435" parent_link="cammera_connect" rate="10">
+    <origin xyz="0.001 -0.07 0.0175" rpy="1.5707 -1.5707 0"/>
+  </xacro:realsense_d435>
+    <link name="gripper_connect">
+        <visual>
+            <geometry>
+                <cylinder radius="${force_sensor_radius}" length="0.1" />
+            </geometry>
+            <origin xyz="0.0 0.0 0.0" rpy="0 0.0 0.0"/>
+            <material name="yellow">
+                <color rgba="0 0.3 0.0 0.5" />
             </material>
         </visual>
@@ -32,8 +120,15 @@
         <xacro:cylinder_inertial_matrix m="${force_sensor_mass}" r="${force_sensor_radius}" h="${force_sensor_h}" />
     </link>
-    <joint name="ft_sensor_joint" type="fixed">
-        <origin xyz="0.0 0 0.0" rpy="0 0.0 0.0"/>
-        <parent link="wrist_3"/>
-        <child link="ft_sensor"/>
+    <joint name="gripper_connect_joint" type="fixed">
+        <origin xyz="0.0 0 0.014" rpy="0 0.0 0.0"/>
+        <parent link="ft_sensor"/>
+        <child link="gripper_connect"/>
+        <axis xyz="0.0 0.0 0.0"/>
+        <limit effort="140.0" lower="${-pi}" upper="${pi}" velocity="${165*pi/180}"/>
+    </joint>
+    <joint name="gripper_connect" type="fixed">
+        <origin xyz="0.0 0 0.0501" rpy="0 0.0 0.0"/>
+        <parent link="gripper_connect"/>
+        <child link="robotiq_arg2f_base_link"/>
         <axis xyz="0.0 0.0 0.0"/>
         <limit effort="140.0" lower="${-pi}" upper="${pi}" velocity="${165*pi/180}"/>
@@ -51,3 +146,40 @@
         </plugin>
     </gazebo>
+        <!-- <gazebo reference="camera_link">
+      <sensor type="depth" name="camera">
+        <always_on>true</always_on>
+        <update_rate>20.0</update_rate>
+        <camera>
+          <horizontal_fov>${60.0*PI/180.0}</horizontal_fov>
+          <image>
+            <format>R8G8B8</format>
+            <width>640</width>
+            <height>480</height>
+          </image>
+          <clip>
+            <near>0.05</near>
+            <far>16.0</far>
+          </clip>
+        </camera>
+        <plugin name="kinect_camera_controller" filename="libgazebo_ros_openni_kinect.so">
+          <cameraName>camera</cameraName>
+          <alwaysOn>true</alwaysOn>
+          <updateRate>10</updateRate>
+          <imageTopicName>rgb/image_raw</imageTopicName>
+          <depthImageTopicName>depth/image_raw</depthImageTopicName>
+          <pointCloudTopicName>depth/points</pointCloudTopicName>
+          <cameraInfoTopicName>rgb/camera_info</cameraInfoTopicName>
+          <depthImageCameraInfoTopicName>depth/camera_info</depthImageCameraInfoTopicName>
+          <frameName>camera_link</frameName>
+          <baseline>0.1</baseline>
+          <distortion_k1>0.0</distortion_k1>
+          <distortion_k2>0.0</distortion_k2>
+          <distortion_k3>0.0</distortion_k3>
+          <distortion_t1>0.0</distortion_t1>
+          <distortion_t2>0.0</distortion_t2>
+          <pointCloudCutoff>0.4</pointCloudCutoff>
+        </plugin>
+      </sensor>
+    </gazebo>
+ -->
 </robot>

Commit message: 夹取方块成功，测试版1

File: sia_manipulator_description/urdf/sia_maipulator_with_force_sensor.xacro (robot description, xacro)
@@ -4,6 +4,7 @@
   <xacro:arg name="use_nominal_extrinsics" default="true"/>
   <xacro:include filename="$(find sia_manipulator_description)/urdf/_d455.urdf.xacro" />
-   <xacro:include filename="$(find sia_manipulator_description)/urdf/robotiq_arg2f_85_model_macro.xacro" />
-  <xacro:robotiq_arg2f_85 prefix=""/>
+   <!-- <xacro:include filename="$(find sia_manipulator_description)/urdf/robotiq_arg2f_85_model_macro.xacro" />
+  <xacro:robotiq_arg2f_85 prefix=""/> -->
+    <xacro:include filename="$(find sia_manipulator_description)/urdf/robotiq_85_gripper.urdf.xacro" />
     <xacro:include filename="$(find sia_manipulator_description)/urdf/depthcam.xacro"/>
   <xacro:include filename="$(find sia_manipulator_description)/urdf/sia_manipulator.xacro" />
@@ -127,5 +128,5 @@
         <limit effort="140.0" lower="${-pi}" upper="${pi}" velocity="${165*pi/180}"/>
     </joint>
-    <joint name="gripper_connect" type="fixed">
+    <!-- <joint name="gripper_connect" type="fixed">
         <origin xyz="0.0 0 0.0501" rpy="0 0 0.0"/>
         <parent link="gripper_connect"/>
@@ -133,5 +134,8 @@
         <axis xyz="0.0 0.0 0.0"/>
         <limit effort="140.0" lower="${-pi}" upper="${pi}" velocity="${165*pi/180}"/>
-    </joint>
+    </joint> -->
+    <xacro:robotiq_85_gripper prefix="" parent="gripper_connect" >
+        <origin xyz="0 0 0.0501" rpy="0 -1.5707 0"/>
+    </xacro:robotiq_85_gripper>
     <gazebo reference="ft_sensor_joint">
         <provideFeedback>true</provideFeedback>
@@ -183,3 +187,26 @@
     </gazebo>
  -->
+ <!--
+     简单测试夹取
+  -->
+  <gazebo>
+   <plugin name="gazebo_grasp_fix" filename="libgazebo_grasp_fix.so">
+        <arm>
+           <arm_name>sia_manipulator_with_force_sensor_gripper</arm_name>
+           <!--与夹持器末端 link 相连的 link 、,可以配置多个-->
+                <palm_link>robotiq_85_left_inner_knuckle_link</palm_link>
+                <!--直接与抓取物体接触的 link ,与 palm_link 之间不能存在其他的 link-->
+                <gripper_link>robotiq_85_left_finger_tip_link</gripper_link>
+                <palm_link>robotiq_85_right_inner_knuckle_link</palm_link>
+                <gripper_link>robotiq_85_right_finger_tip_link</gripper_link>
+        </arm>
+       <forces_angle_tolerance>150</forces_angle_tolerance>
+       <update_rate>130</update_rate>
+       <grip_count_threshold>2</grip_count_threshold>
+       <max_grip_count>8</max_grip_count>
+       <release_tolerance>0.01</release_tolerance>
+       <disable_collisions_on_attach>true</disable_collisions_on_attach>
+       <contact_topic>__default_topic__</contact_topic>
+    </plugin>
+</gazebo>
 </robot>
