Commit message: add the force sensor + fix the previous bug

File: sia_manipulator_simulation/urdf/sia.gazebo.xacro (robot description, xacro)
@@ -23,4 +23,12 @@
       <selfCollide>true</selfCollide>
     </gazebo> -->
+    <!-- <gazebo reference="ft_sensor">
+      <selfCollide>true</selfCollide>
+    </gazebo>
+    <gazebo reference="ft_sensor_joint">
+        <material>Gazebo/Blue</material>
+        <provideFeedback>true</provideFeedback>
+        <disableFixedJointLumping>true</disableFixedJointLumping>
+    </gazebo> -->
   </xacro:macro>
 </robot>

File: sia_manipulator_simulation/urdf/sia.transmission.xacro (robot description, xacro)
@@ -56,4 +56,13 @@
       </actuator>
     </transmission>
+    <!-- <transmission name="ft_sensor_trans">
+      <type>transmission_interface/SimpleTransmission</type>
+      <joint name="ft_sensor_joint">
+        <hardwareInterface>${hw_interface}</hardwareInterface>
+      </joint>
+      <actuator name="ft_sensor_motor">
+        <mechanicalReduction>1</mechanicalReduction>
+      </actuator>
+    </transmission> -->
   </xacro:macro>
 </robot>

File: sia_manipulator_simulation/urdf/sia_manipulator_gazebo.urdf.xacro (robot description, xacro)
@@ -7,5 +7,6 @@
   <xacro:include filename="$(find sia_manipulator_simulation)/urdf/sia.gazebo.xacro" />
   <xacro:include filename="$(find sia_manipulator_simulation)/urdf/sia.transmission.xacro" />
-  <xacro:include filename="$(find sia_manipulator_description)/urdf/sia_manipulator.xacro" />
+  <xacro:include filename="$(find sia_manipulator_description)/urdf/sia_maipulator_with_force_sensor.xacro" />
+  <!-- <xacro:include filename="$(find sia_manipulator_description)/urdf/sia_manipulator.xacro" /> -->
   <!-- arm -->
   <xacro:sia_gazebo  flag="-1"  />

File: sia_robot_description/urdf/sia_robot.xacro (robot description, xacro)
@@ -4,6 +4,7 @@
   <xacro:arg name="transmission_hw_interface" default="hardware_interface/PositionJointInterface"/>
     <!-- arm -->
-  <xacro:include filename="$(find sia_manipulator_description)/urdf/sia_manipulator.xacro" />
-  <xacro:include filename="$(find sia_agv_description)/urdf/sia_agv.urdf.xacro" />
+  <!-- <xacro:include filename="$(find sia_manipulator_description)/urdf/sia_manipulator.xacro" /> -->
+   <xacro:include filename="$(find sia_manipulator_description)/urdf/sia_maipulator_with_force_sensor.xacro" />
+  <xacro:include filename="$(find sia_agv_description)/urdf/sia_agv_on_rviz.urdf.xacro" />
   <joint name="connect_joint" type="fixed">
     <origin xyz="0 0 -0.01" rpy="0 0 0" />
